Commit message: Added controllers and driver launch script

File: jedgar_description/urdf/jedgar.urdf.xacro (robot description, xacro)
@@ -16,4 +16,10 @@
                 </geometry>
             </visual>
+            <collision>
+                <origin rpy="${pi/2} 0 0"/>
+                <geometry>
+                    <cylinder length="${WHEEL_THICKNESS}" radius="${WHEEL_RADIUS}"/>
+                </geometry>
+            </collision>
         </link>
     </xacro:macro>

Commit message: Gazeboified Jedgar description

File: jedgar_description/urdf/jedgar.urdf.xacro (robot description, xacro)
@@ -1,11 +1,19 @@
 <?xml version="1.0"?>
 <robot xmlns:xacro="http://www.ros.org/wiki/xacro" name="jedgar">
+    <gazebo>
+        <plugin name="gazebo_ros_control" filename="libgazebo_ros_control.so">
+            <robotSimType>gazebo_ros_control/DefaultRobotHWSim</robotSimType>
+        </plugin>
+    </gazebo>
     <!-- TODO Measure Jedgar -->
     <xacro:property name="BASE_LENGTH" value="1.0" />
     <xacro:property name="BASE_HEIGHT" value="1.0" />
+    <xacro:property name="BASE_MASS" value="1.0" />
     <xacro:property name="WHEEL_TO_BACK" value="1.0" />
     <xacro:property name="WHEELBASE" value="1.0" />
     <xacro:property name="WHEEL_THICKNESS" value="1.0" />
     <xacro:property name="WHEEL_RADIUS" value="1.0" />
+    <xacro:property name="WHEEL_MASS" value="1.0" />
+    <xacro:property name="WHEEL_MOMENT" value="${WHEEL_MASS/12*(3*WHEEL_RADIUS**2+WHEEL_THICKNESS**2)}" />
     <xacro:macro name="wheel" params="name">
         <link name="${name}">
@@ -22,4 +30,8 @@
                 </geometry>
             </collision>
+            <inertial>
+                <mass value="${WHEEL_MASS}"/>
+                <inertia ixx="${WHEEL_MOMENT}" iyy="${WHEEL_MOMENT}" izz="${WHEEL_MOMENT}" ixy="0" ixz="0" iyz="0"/>
+            </inertial>
         </link>
     </xacro:macro>
@@ -31,4 +43,17 @@
             </geometry>
         </visual>
+        <collision>
+            <geometry>
+                <box size="${BASE_LENGTH} ${WHEELBASE} ${BASE_HEIGHT}"/>
+            </geometry>
+        </collision>
+        <inertial>
+            <mass value="${BASE_MASS}"/>
+            <inertia
+                ixx="${BASE_MASS/12*(BASE_HEIGHT**2+BASE_LENGTH**2)}"
+                iyy="${BASE_MASS/12*(WHEELBASE**2+BASE_LENGTH**2)}"
+                izz="${BASE_MASS/12*(WHEELBASE**2+BASE_HEIGHT**2)}"
+                ixy="0" ixz="0" iyz="0"/>
+        </inertial>
     </link>
     <xacro:wheel name="left_wheel"/>
@@ -45,4 +70,14 @@
         <origin xyz="${-BASE_LENGTH/2+WHEEL_TO_BACK} ${WHEELBASE/2} 0"/>
     </joint>
+    <transmission name="left_wheel_transmission">
+        <type>transmission_interface/SimpleTransmission</type>
+        <joint name="left_wheel_joint">
+            <hardwareInterface>hardware_interface/VelocityJointInterface</hardwareInterface>
+        </joint>
+        <actuator name="left_motor">
+            <hardwareInterface>hardware_interface/VelocityJointInterface</hardwareInterface>
+            <mechanicalReduction>1</mechanicalReduction>
+        </actuator>
+    </transmission>
     <joint name="right_wheel_joint" type="continuous">
         <parent link="base_link"/>
@@ -51,3 +86,13 @@
         <origin xyz="${-BASE_LENGTH/2+WHEEL_TO_BACK} ${-WHEELBASE/2} 0"/>
     </joint>
+    <transmission name="right_wheel_transmission">
+        <type>transmission_interface/SimpleTransmission</type>
+        <joint name="right_wheel_joint">
+            <hardwareInterface>hardware_interface/VelocityJointInterface</hardwareInterface>
+        </joint>
+        <actuator name="right_motor">
+            <hardwareInterface>hardware_interface/VelocityJointInterface</hardwareInterface>
+            <mechanicalReduction>1</mechanicalReduction>
+        </actuator>
+    </transmission>
 </robot>

Commit message: Added dimension estimates

File: jedgar_description/urdf/jedgar.urdf.xacro (robot description, xacro)
@@ -7,11 +7,11 @@
     </gazebo>
     <!-- TODO Measure Jedgar -->
-    <xacro:property name="BASE_LENGTH" value="1.0" />
-    <xacro:property name="BASE_HEIGHT" value="1.0" />
+    <xacro:property name="BASE_LENGTH" value="0.300" />
+    <xacro:property name="BASE_HEIGHT" value="0.050" />
     <xacro:property name="BASE_MASS" value="1.0" />
-    <xacro:property name="WHEEL_TO_BACK" value="1.0" />
-    <xacro:property name="WHEELBASE" value="1.0" />
-    <xacro:property name="WHEEL_THICKNESS" value="1.0" />
-    <xacro:property name="WHEEL_RADIUS" value="1.0" />
+    <xacro:property name="WHEEL_THICKNESS" value="0.020" />
+    <xacro:property name="WHEEL_RADIUS" value="0.075" />
+    <xacro:property name="WHEEL_TO_BACK" value="${WHEEL_RADIUS}" />
+    <xacro:property name="WHEELBASE" value="0.200" />
     <xacro:property name="WHEEL_MASS" value="1.0" />
     <xacro:property name="WHEEL_MOMENT" value="${WHEEL_MASS/12*(3*WHEEL_RADIUS**2+WHEEL_THICKNESS**2)}" />
@@ -57,4 +57,22 @@
         </inertial>
     </link>
+    <link name="caster_link">
+        <visual>
+            <geometry>
+                <sphere radius="0.01"/>
+            </geometry>
+        </visual>
+        <collision>
+            <geometry>
+                <sphere radius="0.01"/>
+            </geometry>
+        </collision>
+        <inertial>
+            <mass value="0"/>
+            <inertia
+                ixx="0" iyy="0" izz="0"
+                ixy="0" ixz="0" iyz="0"/>
+        </inertial>
+    </link>
     <xacro:wheel name="left_wheel"/>
     <xacro:wheel name="right_wheel"/>
@@ -62,5 +80,10 @@
         <parent link="base_link"/>
         <child link="base_footprint"/>
-        <origin xyz="0 0 ${WHEEL_RADIUS}"/>
+        <origin xyz="0 0 ${-WHEEL_RADIUS}"/>
+    </joint>
+    <joint name="caster_joint" type="fixed">
+        <parent link="base_link"/>
+        <child link="caster_link"/>
+        <origin xyz="${BASE_LENGTH/2} 0 ${-WHEEL_RADIUS + 0.01}"/>
     </joint>
     <joint name="left_wheel_joint" type="continuous">

Commit message: Added more gazebo sensors

File: jedgar_description/urdf/jedgar.urdf.xacro (robot description, xacro)
@@ -1,9 +1,5 @@
 <?xml version="1.0"?>
 <robot xmlns:xacro="http://www.ros.org/wiki/xacro" name="jedgar">
-    <gazebo>
-        <plugin name="gazebo_ros_control" filename="libgazebo_ros_control.so">
-            <robotSimType>gazebo_ros_control/DefaultRobotHWSim</robotSimType>
-        </plugin>
-    </gazebo>
+    <xacro:include filename="$(find jedgar_description)/urdf/jedgar.gazebo" />
     <!-- TODO Measure Jedgar -->
     <xacro:property name="BASE_LENGTH" value="0.300" />
@@ -16,4 +12,5 @@
     <xacro:property name="WHEEL_MASS" value="1.0" />
     <xacro:property name="WHEEL_MOMENT" value="${WHEEL_MASS/12*(3*WHEEL_RADIUS**2+WHEEL_THICKNESS**2)}" />
+    <xacro:property name="camera_link" value="0.005" />
     <xacro:macro name="wheel" params="name">
         <link name="${name}">
@@ -75,4 +72,28 @@
         </inertial>
     </link>
+	<link name="camera_link">
+		<collision>
+			<origin xyz="0 0 0" rpy="0 0 0"/>
+			<geometry>
+				<box size="${camera_link} ${camera_link} ${camera_link}"/>
+			</geometry>
+		</collision>
+		<visual>
+			<origin xyz="0 0 0" rpy="0 0 0"/>
+			<geometry>
+		<box size="${camera_link} ${camera_link} ${camera_link}"/>
+			</geometry>
+		</visual>
+		<inertial>
+			<mass value="1e-5" />
+			<origin xyz="0 0 0" rpy="0 0 0"/>
+			<inertia ixx="1e-6" ixy="0" ixz="0" iyy="1e-6" iyz="0" izz="1e-6" />
+		</inertial>
+	</link>
+    <joint name="camera_joint" type="fixed">
+        <parent link="base_link"/>
+        <child link="camera_link"/>
+        <origin xyz="${BASE_LENGTH/2} 0 0"/>
+    </joint>
     <xacro:wheel name="left_wheel"/>
     <xacro:wheel name="right_wheel"/>

Commit message: Added navigation laser and lost weight

File: jedgar_description/urdf/jedgar.urdf.xacro (robot description, xacro)
@@ -5,12 +5,13 @@
     <xacro:property name="BASE_LENGTH" value="0.300" />
     <xacro:property name="BASE_HEIGHT" value="0.050" />
-    <xacro:property name="BASE_MASS" value="1.0" />
+    <xacro:property name="BASE_MASS" value="0.4" />
     <xacro:property name="WHEEL_THICKNESS" value="0.020" />
     <xacro:property name="WHEEL_RADIUS" value="0.075" />
     <xacro:property name="WHEEL_TO_BACK" value="${WHEEL_RADIUS}" />
     <xacro:property name="WHEELBASE" value="0.200" />
-    <xacro:property name="WHEEL_MASS" value="1.0" />
+    <xacro:property name="WHEEL_MASS" value="0.1" />
     <xacro:property name="WHEEL_MOMENT" value="${WHEEL_MASS/12*(3*WHEEL_RADIUS**2+WHEEL_THICKNESS**2)}" />
     <xacro:property name="camera_link" value="0.005" />
+    <xacro:property name="laser_link" value="0.1" />
     <xacro:macro name="wheel" params="name">
         <link name="${name}">
@@ -96,4 +97,29 @@
         <origin xyz="${BASE_LENGTH/2} 0 0"/>
     </joint>
+	<link name="laser_link">
+		<collision>
+			<origin xyz="0 0 0" rpy="0 0 0"/>
+			<geometry>
+				<box size="${laser_link} ${laser_link} ${laser_link}"/>
+			</geometry>
+		</collision>
+		<visual>
+			<origin xyz="0 0 0" rpy="0 0 0"/>
+			<geometry>
+		<box size="${laser_link} ${laser_link} ${laser_link}"/>
+			</geometry>
+		</visual>
+		<inertial>
+			<mass value="1e-5" />
+			<origin xyz="0 0 0" rpy="0 0 0"/>
+			<inertia ixx="1e-6" ixy="0" ixz="0" iyy="1e-6" iyz="0" izz="1e-6" />
+		</inertial>
+	</link>
+    <joint name="laser_joint" type="fixed">
+        <parent link="base_link"/>
+        <child link="laser_link"/>
+        <origin xyz="${BASE_LENGTH/2} ${-WHEELBASE/2} 0"
+				rpy="0 0 0"/>
+    </joint>
     <xacro:wheel name="left_wheel"/>
     <xacro:wheel name="right_wheel"/>
